File: chasma.kicad_pcb (KiCad board)
At the start: 2 copper layers, 366 x 181.5 mm, 186 parts, among them J0 USB_C_Receptacle_USB2.0, SW00_00 SW_Push, SW00_01 SW_Push, SW00_02 SW_Push, SW00_03 SW_Push, SW01_00 SW_Push, SW01_01 SW_Push, SW01_02 SW_Push, SW01_03 SW_Push, SW02_00 SW_Push, SW02_01 SW_Push, SW02_02 SW_Push, SW02_03 SW_Push, SW03_00 SW_Push, SW03_01 SW_Push, SW03_02 SW_Push, SW03_03 SW_Push, SW04_00 SW_Push, SW04_01 SW_Push, SW04_02 SW_Push, SW05_00 SW_Push, SW05_01 SW_Push, SW05_02 SW_Push, SW05_03 SW_Push, SW06_00 SW_Push, SW06_01 SW_Push, SW06_02 SW_Push, SW07_00 SW_Push, SW07_01 SW_Push, SW07_02 SW_Push, SW07_03 SW_Push, SW08_00 SW_Push, SW08_01 SW_Push, SW08_02 SW_Push, SW09_00 SW_Push, SW09_01 SW_Push, SW09_02 SW_Push, SW09_03 SW_Push, SW10_00 SW_Push, SW10_01 SW_Push, SW10_02 SW_Push, SW10_03 SW_Push, SW11_00 SW_Push, SW11_01 SW_Push, SW11_02 SW_Push, SW12_00 SW_Push, SW12_01 SW_Push, SW12_03 SW_Push, SW13_00 SW_Push, SW13_02 SW_Push, SW13_03 SW_Push, SW14_00 SW_Push, SW14_01 SW_Push, SW14_03 SW_Push, U0 ATmega32U4-A, Y0 16Mhz

Commit message: initial pcb
Parts:
- moved LED00_03 296.5 mm to (65.6, 208.4)
- moved LED01_03 277.4 mm to (89.4, 208.4)
- moved LED02_03 265.7 mm to (113.2, 208.4)
- moved D14_01 257.7 mm to (355.9, 170.4), turned to 90 degrees
- moved ULED00 238.5 mm to (339.5, 134.6), turned to -90 degrees
- moved LED01_00 229.7 mm to (91.8, 151.3)
- moved LED00_02 224.5 mm to (75.0, 189.4)
- moved LED03_02 222.9 mm to (144.1, 189.4)
- moved LED02_01 220.2 mm to (115.6, 170.3)
- moved D14_00 218.4 mm to (355.9, 151.3), turned to 90 degrees
- moved LED00_00 216.2 mm to (68.0, 151.3)
- moved LED04_02 215.7 mm to (163.2, 189.4)
- moved LED03_03 215.6 mm to (146.5, 208.4)
- moved LED01_02 215.5 mm to (106.0, 189.4)
- moved D12_03 212.9 mm to (317.9, 208.5), turned to 90 degrees
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
Commit message: add case
Parts:
- moved J0 0.95 mm to (206.0, 132.8)
Other:
- board size 366 x 181.5 mm -> 304.8 x 83.1 mm
Changed lines of the file:
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@@
   )
   (footprint "Connector_USB:USB_C_Receptacle_HRO_TYPE-C-31-M-12" (layer "B.Cu")
-    (at 206 131.85)
+    (at 206 132.8)
     (descr "USB Type-C receptacle for USB 2.0 and PD, http://www.krhro.com/uploads/soft/180320/1-1P320120243.pdf")
     (tags "usb usb-c 2.0 pd")
@@
   (gr_line (start 208.310014 177.8) (end 208.310014 191.8) (layer "Eco1.User") (width 0.1))
   (gr_line (start 317.846986 210.850003) (end 317.846986 210.850003) (layer "Eco1.User") (width 0.1))
-  (gr_line (start 389.15 49.9) (end 27.6 52.9) (layer "Edge.Cuts") (width 0.1))
-  (gr_line (start 23.1 231.4) (end 389.15 229.9) (layer "Edge.Cuts") (width 0.1))
-  (gr_line (start 27.6 52.9) (end 23.1 231.4) (layer "Edge.Cuts") (width 0.1))
-  (gr_line (start 389.15 229.9) (end 389.15 49.9) (layer "Edge.Cuts") (width 0.1))
+  (gr_poly
+    (pts
+      (xy 210.523328 130.275668)
+      (xy 210.710965 130.333953)
+      (xy 210.880734 130.426172)
+      (xy 211.028607 130.548299)
+      (xy 211.150586 130.696307)
+      (xy 211.242688 130.866169)
+      (xy 211.300794 131.053857)
+      (xy 211.320889 131.255345)
+      (xy 211.320264 131.870302)
+      (xy 211.319638 132.485259)
+      (xy 211.319013 133.100217)
+      (xy 211.317136 134.94509)
+      (xy 211.31651 135.560048)
+      (xy 211.315885 136.175006)
+      (xy 211.33598 136.376493)
+      (xy 211.394086 136.564181)
+      (xy 211.486188 136.734041)
+      (xy 211.608151 136.882048)
+      (xy 211.75604 137.004175)
+      (xy 211.925809 137.096393)
+      (xy 212.113431 137.154677)
+      (xy 212.314817 137.174999)
+      (xy 230.447507 137.174894)
+      (xy 266.712857 137.174684)
+      (xy 284.845548 137.174579)
+      (xy 302.978223 137.174475)
+      (xy 321.110898 137.17437)
+      (xy 357.376279 137.17416)
+      (xy 357.577817 137.194475)
+      (xy 357.765531 137.252743)
+      (xy 357.935391 137.344941)
+      (xy 358.083402 137.467049)
+      (xy 358.205503 137.615045)
+      (xy 358.297696 137.784909)
+      (xy 358.355985 137.972619)
+      (xy 358.376279 138.174153)
+      (xy 358.376279 212.34935)
+      (xy 358.355985 212.550888)
+      (xy 358.297696 212.738601)
+      (xy 358.205503 212.90847)
+      (xy 358.083402 213.056465)
+      (xy 357.935391 213.178573)
+      (xy 357.765531 213.270775)
+      (xy 357.577817 213.329048)
+      (xy 357.376279 213.349365)
+      (xy 54.613962 213.349365)
+      (xy 54.412427 213.329033)
+      (xy 54.224717 213.270759)
+      (xy 54.054853 213.178558)
+      (xy 53.906855 213.05645)
+      (xy 53.784746 212.908455)
+      (xy 53.692547 212.738586)
+      (xy 53.634278 212.55088)
+      (xy 53.613962 212.349342)
+      (xy 53.613962 138.174155)
+      (xy 53.634278 137.97262)
+      (xy 53.692547 137.78491)
+      (xy 53.784747 137.615047)
+      (xy 53.906856 137.46705)
+      (xy 54.054853 137.344942)
+      (xy 54.224717 137.252744)
+      (xy 54.412427 137.194476)
+      (xy 54.613962 137.174161)
+      (xy 72.746593 137.174266)
+      (xy 90.879224 137.174371)
+      (xy 109.011853 137.174475)
+      (xy 127.144483 137.174581)
+      (xy 145.277112 137.174685)
+      (xy 199.675 137.175)
+      (xy 199.876599 137.154691)
+      (xy 200.064405 137.09644)
+      (xy 200.234357 137.004262)
+      (xy 200.382474 136.882172)
+      (xy 200.504712 136.734187)
+      (xy 200.597012 136.56432)
+      (xy 200.655408 136.376588)
+      (xy 200.6759 136.175007)
+      (xy 200.676526 135.560049)
+      (xy 200.677152 134.945091)
+      (xy 200.677777 134.330133)
+      (xy 200.68028 131.870303)
+      (xy 200.680905 131.255345)
+      (xy 200.701398 131.053763)
+      (xy 200.759793 130.866031)
+      (xy 200.852201 130.696164)
+      (xy 200.974439 130.548177)
+      (xy 201.122556 130.426087)
+      (xy 201.292508 130.333908)
+      (xy 201.480298 130.275655)
+      (xy 201.682019 130.255345)
+      (xy 210.321851 130.255345)
+    ) (layer "Edge.Cuts") (width 0.2) (fill none))
+  (group "" (id c96b22e8-ed17-431f-9fa1-197cd577573a)
+    (members
+      cbd2b97a-bfcd-48ad-95dd-b02946f2bc71
+    )
+  )
 )
