File: chasma.kicad_sch (KiCad schematic)
At the start: 123 parts, among them J0 USB_C_Receptacle_USB2.0, SW00_00 SW_Push, SW00_01 SW_Push, SW00_02 SW_Push, SW00_03 SW_Push, SW01_00 SW_Push, SW01_01 SW_Push, SW01_02 SW_Push, SW01_03 SW_Push, SW02_00 SW_Push, SW02_01 SW_Push, SW02_02 SW_Push, SW02_03 SW_Push, SW03_00 SW_Push, SW03_01 SW_Push, SW03_02 SW_Push, SW03_03 SW_Push, SW04_00 SW_Push, SW04_01 SW_Push, SW04_02 SW_Push, SW05_00 SW_Push, SW05_01 SW_Push, SW05_02 SW_Push, SW05_03 SW_Push, SW06_00 SW_Push, SW06_01 SW_Push, SW06_02 SW_Push, SW07_00 SW_Push, SW07_01 SW_Push, SW07_02 SW_Push, SW07_03 SW_Push, SW08_00 SW_Push, SW08_01 SW_Push, SW08_02 SW_Push, SW09_00 SW_Push, SW09_01 SW_Push, SW09_02 SW_Push, SW09_03 SW_Push, SW10_00 SW_Push, SW10_01 SW_Push, SW10_02 SW_Push, SW10_03 SW_Push, SW11_00 SW_Push, SW11_01 SW_Push, SW11_02 SW_Push, SW12_00 SW_Push, SW12_01 SW_Push, SW12_03 SW_Push, SW13_00 SW_Push, SW13_02 SW_Push, SW13_03 SW_Push, SW14_00 SW_Push, SW14_01 SW_Push, SW14_03 SW_Push, U0 ATmega32U4-A, Y0 16Mhz

Commit message: wip
Parts:
- added LED00_00, LED00_01, LED00_02, LED00_03, LED01_00, LED01_01, LED01_02, LED01_03, LED02_00, LED02_01, LED02_02, LED02_03, LED03_00, LED03_01, LED03_02, LED03_03, LED04_00, LED04_01, LED04_02, LED05_00, LED05_01, LED05_02, LED05_03, LED06_00, LED06_01, LED06_02, LED07_00, LED07_01, LED07_02, LED07_03, LED08_00, LED08_01, LED08_02, LED09_00, LED09_01, LED09_02, LED09_03, LED10_00, LED10_01, LED10_02, LED10_03, LED11_00, LED11_01, LED11_02, LED12_00, LED12_01, LED12_03, LED13_00, LED13_02, LED13_03, LED14_00, LED14_01, LED14_03: SK6812MINI-E, SK6812MINI-E:SK6812MINIE, symbol SK6812MINI-E:SK6812MINI-E
- added ULED00, ULED01, ULED02, ULED03, ULED04, ULED05, ULED06, ULED07, ULED08, ULED09: WS2812B, WS2812B:WS2812B, symbol ws2812b:WS2812B
- SW00_00, SW13_00: footprint MX_Only:MXOnly-1U-Hotswap -> MX_Only:MXOnly-1.5U-Hotswap
- SW00_01: footprint MX_Only:MXOnly-1.5U-Hotswap -> MX_Only:MXOnly-1.75U-Hotswap
- SW00_02: footprint MX_Only:MXOnly-1.25U-Hotswap -> MX_Only:MXOnly-2.25U-Hotswap
- SW01_01, SW02_01, SW03_01, SW04_01, SW05_01, SW06_01, SW07_01, SW08_01, SW09_01, SW10_01, SW11_01, SW14_01: footprint MX_Only:MXOnly-1.5U-Hotswap -> MX_Only:MXOnly-1U-Hotswap
- SW01_02, SW02_02, SW03_02, SW04_02, SW05_02, SW06_02, SW07_02, SW08_02, SW09_02, SW10_02, SW12_03, SW13_02, SW13_03, SW14_03: footprint MX_Only:MXOnly-1.25U-Hotswap -> MX_Only:MXOnly-1U-Hotswap
- SW03_03: footprint MX_Only:MXOnly-1.25U-Hotswap -> MX_Only:MXOnly-2.25U-Hotswap-ReversedStabilizers
- SW07_03: footprint MX_Only:MXOnly-1.25U-Hotswap -> MX_Only:MXOnly-2.75U-Hotswap-ReversedStabilizers
- SW11_02: footprint MX_Only:MXOnly-1.25U-Hotswap -> MX_Only:MXOnly-1.75U-Hotswap
- SW12_01: footprint MX_Only:MXOnly-1.5U-Hotswap -> MX_Only:MXOnly-2.25U-Hotswap-ReversedStabilizers
Connections:
- net GND: now also LED00_00.3 (GND), LED00_01.3 (GND), LED00_02.3 (GND), LED00_03.3 (GND), LED01_00.3 (GND), LED01_01.3 (GND), LED01_02.3 (GND), LED01_03.3 (GND), LED02_00.3 (GND), LED02_01.3 (GND), LED02_02.3 (GND), LED02_03.3 (GND), LED03_00.3 (GND), LED03_01.3 (GND), LED03_02.3 (GND), LED03_03.3 (GND), LED04_00.3 (GND), LED04_01.3 (GND), LED04_02.3 (GND), LED05_00.3 (GND), LED05_01.3 (GND), LED05_02.3 (GND), LED05_03.3 (GND), LED06_00.3 (GND), LED06_01.3 (GND), LED06_02.3 (GND), LED07_00.3 (GND), LED07_01.3 (GND), LED07_02.3 (GND), LED07_03.3 (GND), LED08_00.3 (GND), LED08_01.3 (GND), LED08_02.3 (GND), LED09_00.3 (GND), LED09_01.3 (GND), LED09_02.3 (GND), LED09_03.3 (GND), LED10_00.3 (GND), LED10_01.3 (GND), LED10_02.3 (GND), LED10_03.3 (GND), LED11_00.3 (GND), LED11_01.3 (GND), LED11_02.3 (GND), LED12_00.3 (GND), LED12_01.3 (GND), LED12_03.3 (GND), LED13_00.3 (GND), LED13_02.3 (GND), LED13_03.3 (GND), LED14_00.3 (GND), LED14_01.3 (GND), LED14_03.3 (GND), ULED00.3 (GND), ULED01.3 (GND), ULED02.3 (GND), ULED03.3 (GND), ULED04.3 (GND), ULED05.3 (GND), ULED06.3 (GND), ULED07.3 (GND), ULED08.3 (GND), ULED09.3 (GND)
- net LED: now also LED00_03.4 (DIN)
- net VCC: now also LED00_00.1 (VDD), LED00_01.1 (VDD), LED00_02.1 (VDD), LED00_03.1 (VDD), LED01_00.1 (VDD), LED01_01.1 (VDD), LED01_02.1 (VDD), LED01_03.1 (VDD), LED02_00.1 (VDD), LED02_01.1 (VDD), LED02_02.1 (VDD), LED02_03.1 (VDD), LED03_00.1 (VDD), LED03_01.1 (VDD), LED03_02.1 (VDD), LED03_03.1 (VDD), LED04_00.1 (VDD), LED04_01.1 (VDD), LED04_02.1 (VDD), LED05_00.1 (VDD), LED05_01.1 (VDD), LED05_02.1 (VDD), LED05_03.1 (VDD), LED06_00.1 (VDD), LED06_01.1 (VDD), LED06_02.1 (VDD), LED07_00.1 (VDD), LED07_01.1 (VDD), LED07_02.1 (VDD), LED07_03.1 (VDD), LED08_00.1 (VDD), LED08_01.1 (VDD), LED08_02.1 (VDD), LED09_00.1 (VDD), LED09_01.1 (VDD), LED09_02.1 (VDD), LED09_03.1 (VDD), LED10_00.1 (VDD), LED10_01.1 (VDD), LED10_02.1 (VDD), LED10_03.1 (VDD), LED11_00.1 (VDD), LED11_01.1 (VDD), LED11_02.1 (VDD), LED12_00.1 (VDD), LED12_01.1 (VDD), LED12_03.1 (VDD), LED13_00.1 (VDD), LED13_02.1 (VDD), LED13_03.1 (VDD), LED14_00.1 (VDD), LED14_01.1 (VDD), LED14_03.1 (VDD), ULED00.1 (VCC), ULED01.1 (VCC), ULED02.1 (VCC), ULED03.1 (VCC), ULED04.1 (VCC), ULED05.1 (VCC), ULED06.1 (VCC), ULED07.1 (VCC), ULED08.1 (VCC), ULED09.1 (VCC)
- net row01: now reaches D00_01.1 (K), D01_01.1 (K), D02_01.1 (K), D03_01.1 (K), D04_01.1 (K), D05_01.1 (K), D06_01.1 (K), D07_01.1 (K), D08_01.1 (K), D09_01.1 (K), D10_01.1 (K), D11_01.1 (K), D12_01.1 (K), D14_01.1 (K)
- net row01: now also U0.39 (PF4)
- net row03: now reaches D00_03.1 (K), D01_03.1 (K), D02_03.1 (K), D03_03.1 (K), D05_03.1 (K), D07_03.1 (K), D09_03.1 (K), D10_03.1 (K), D12_03.1 (K), D13_03.1 (K), D14_03.1 (K)
- net row03: now also U0.37 (PF6)
- net row00: now reaches D00_00.1 (K), D01_00.1 (K), D02_00.1 (K), D03_00.1 (K), D04_00.1 (K), D05_00.1 (K), D06_00.1 (K), D07_00.1 (K), D08_00.1 (K), D09_00.1 (K), D10_00.1 (K), D11_00.1 (K), D12_00.1 (K), D13_00.1 (K), D14_00.1 (K)
- net row00: now also U0.40 (PF1)
- net row02: now reaches D00_02.1 (K), D01_02.1 (K), D02_02.1 (K), D03_02.1 (K), D04_02.1 (K), D05_02.1 (K), D06_02.1 (K), D07_02.1 (K), D08_02.1 (K), D09_02.1 (K), D10_02.1 (K), D11_02.1 (K), D13_02.1 (K)
- net row02: now also U0.38 (PF5)
- net col14: now reaches SW14_00.1, SW14_01.1, SW14_03.1
- net col14: now also U0.20 (PD2)
- net col05: now reaches SW05_00.1, SW05_01.1, SW05_02.1, SW05_03.1
- net col05: now also U0.25 (PD4)
- net col10: now reaches SW10_00.1, SW10_01.1, SW10_02.1, SW10_03.1
- net col10: now also U0.12 (PB7)
- net col07: now reaches U0.18 (PD0)
- net col07: now also SW07_00.1, SW07_01.1, SW07_02.1, SW07_03.1
- net col06: now reaches U0.19 (PD1)
- net col06: now also SW06_00.1, SW06_01.1, SW06_02.1
- net col04: now reaches U0.22 (PD5)
- net col04: now also SW04_00.1, SW04_01.1, SW04_02.1
- net col03: now reaches U0.26 (PD6)
- net col03: now also SW03_00.1, SW03_01.1, SW03_02.1, SW03_03.1
- net col02: now reaches U0.27 (PD7)
- net col02: now also SW02_00.1, SW02_01.1, SW02_02.1, SW02_03.1
- net col13: now reaches U0.28 (PB4)
- net col13: now also SW13_00.1, SW13_02.1, SW13_03.1
- net col12: now reaches U0.29 (PB5)
- net col12: now also SW12_00.1, SW12_01.1, SW12_03.1
- net col11: now reaches U0.30 (PB6)
- net col11: now also SW11_00.1, SW11_01.1, SW11_02.1
- net col09: now reaches U0.31 (PC6)
- net col09: now also SW09_00.1, SW09_01.1, SW09_02.1, SW09_03.1
- net col08: now reaches U0.32 (PC7)
- net col08: now also SW08_00.1, SW08_01.1, SW08_02.1
- net col00: now reaches U0.36 (PF7)
- net col00: now also SW00_00.1, SW00_01.1, SW00_02.1, SW00_03.1
- net col01: now reaches U0.41 (PF0)
- net col01: now also SW01_00.1, SW01_01.1, SW01_02.1, SW01_03.1
- new net: ULED00.2 (DOUT), ULED01.4 (DIN)
- new net: LED14_00.2 (DOUT), ULED00.4 (DIN)
- new net: LED12_01.4 (DIN), LED12_03.2 (DOUT)
- new net: LED11_02.2 (DOUT), LED12_03.4 (DIN)
- new net: LED00_00.2 (DOUT), LED01_00.4 (DIN)
- new net: LED00_00.4 (DIN), LED00_01.2 (DOUT)
- new net: LED10_00.4 (DIN), LED10_01.2 (DOUT)
- new net: LED10_01.4 (DIN), LED10_02.2 (DOUT)
- new net: ULED05.2 (DOUT), ULED06.4 (DIN)
- new net: ULED04.2 (DOUT), ULED05.4 (DIN)
- new net: LED02_01.4 (DIN), LED02_02.2 (DOUT)
- new net: LED02_02.4 (DIN), LED02_03.2 (DOUT)
- new net: LED01_01.2 (DOUT), LED01_02.4 (DIN)
- new net: LED01_00.2 (DOUT), LED01_01.4 (DIN)
- new net: LED06_01.4 (DIN), LED06_02.2 (DOUT)
- new net: LED05_03.2 (DOUT), LED06_02.4 (DIN)
- new net: LED10_02.4 (DIN), LED10_03.2 (DOUT)
- new net: LED09_03.2 (DOUT), LED10_03.4 (DIN)
- new net: LED13_00.2 (DOUT), LED13_02.4 (DIN)
- new net: LED12_00.2 (DOUT), LED13_00.4 (DIN)
- new net: LED13_03.2 (DOUT), LED14_03.4 (DIN)
- new net: LED13_02.2 (DOUT), LED13_03.4 (DIN)
- new net: LED12_00.4 (DIN), LED12_01.2 (DOUT)
- new net: LED00_01.4 (DIN), LED00_02.2 (DOUT)
- new net: LED04_00.4 (DIN), LED04_01.2 (DOUT)
- new net: LED04_01.4 (DIN), LED04_02.2 (DOUT)
- new net: LED09_02.2 (DOUT), LED09_03.4 (DIN)
- new net: LED09_01.2 (DOUT), LED09_02.4 (DIN)
- new net: LED05_01.2 (DOUT), LED05_02.4 (DIN)
- new net: LED05_00.2 (DOUT), LED05_01.4 (DIN)
- new net: LED06_00.2 (DOUT), LED07_00.4 (DIN)
- new net: LED06_00.4 (DIN), LED06_01.2 (DOUT)
- new net: ULED01.2 (DOUT), ULED02.4 (DIN)
- new net: LED07_03.2 (DOUT), LED08_02.4 (DIN)
- new net: LED07_02.2 (DOUT), LED07_03.4 (DIN)
- new net: LED08_00.2 (DOUT), LED09_00.4 (DIN)
- new net: LED08_00.4 (DIN), LED08_01.2 (DOUT)
- new net: LED00_02.4 (DIN), LED00_03.2 (DOUT)
- new net: ULED08.2 (DOUT), ULED09.4 (DIN)
- new net: ULED03.2 (DOUT), ULED04.4 (DIN)
- new net: ULED02.2 (DOUT), ULED03.4 (DIN)
- new net: LED09_00.2 (DOUT), LED09_01.4 (DIN)
- new net: LED05_02.2 (DOUT), LED05_03.4 (DIN)
- new net: LED08_01.4 (DIN), LED08_02.2 (DOUT)
- new net: LED14_01.4 (DIN), LED14_03.2 (DOUT)
- new net: LED07_00.2 (DOUT), LED07_01.4 (DIN)
- new net: LED07_01.2 (DOUT), LED07_02.4 (DIN)
- new net: LED10_00.2 (DOUT), LED11_00.4 (DIN)
- new net: LED14_00.4 (DIN), LED14_01.2 (DOUT)
- new net: LED11_01.2 (DOUT), LED11_02.4 (DIN)
- new net: LED03_02.2 (DOUT), LED03_03.4 (DIN)
- new net: LED03_01.2 (DOUT), LED03_02.4 (DIN)
- new net: LED01_02.2 (DOUT), LED01_03.4 (DIN)
- new net: LED03_03.2 (DOUT), LED04_02.4 (DIN)
- new net: LED01_03.2 (DOUT), LED02_03.4 (DIN)
- new net: ULED07.2 (DOUT), ULED08.4 (DIN)
- new net: LED02_00.2 (DOUT), LED03_00.4 (DIN)
- new net: LED02_00.4 (DIN), LED02_01.2 (DOUT)
- new net: LED04_00.2 (DOUT), LED05_00.4 (DIN)
- new net: LED03_00.2 (DOUT), LED03_01.4 (DIN)
- new net: LED11_00.2 (DOUT), LED11_01.4 (DIN)
- new net: ULED06.2 (DOUT), ULED07.4 (DIN)
- no-connect marks 3 -> 9
Other:
- title: (none) -> chasma

Commit message: create pcb
Parts:
- added ULED10, ULED11: WS2812B, WS2812B:WS2812B, symbol ws2812b:WS2812B
Connections:
- net GND: now also ULED10.3 (GND), ULED11.3 (GND)
- net VCC: now also ULED10.1 (VCC), ULED11.1 (VCC)
- net col00: now also U0.26 (PD6); no longer U0.36 (PF7)
- net col01: now also U0.27 (PD7); no longer U0.41 (PF0)
- net col02: now also U0.28 (PB4); no longer U0.27 (PD7)
- net col03: now also U0.29 (PB5); no longer U0.26 (PD6)
- net col04: now also U0.30 (PB6); no longer U0.22 (PD5)
- net col05: now also U0.31 (PC6); no longer U0.25 (PD4)
- net col06: now also U0.39 (PF4); no longer U0.19 (PD1)
- net col07: now also U0.40 (PF1); no longer U0.18 (PD0)
- net col08: now also U0.1 (PE6); no longer U0.32 (PC7)
- net col09: now also U0.8 (PB0); no longer U0.31 (PC6)
- net col10: now also U0.9 (PB1); no longer U0.12 (PB7)
- net col11: now also U0.10 (PB2); no longer U0.30 (PB6)
- net col12: now also U0.11 (PB3); no longer U0.29 (PB5)
- net col13: now also U0.12 (PB7); no longer U0.28 (PB4)
- net col14: now also U0.18 (PD0); no longer U0.20 (PD2)
- net row00: now also U0.38 (PF5); no longer U0.40 (PF1)
- net row01: now also U0.37 (PF6); no longer U0.39 (PF4)
- net row02: now also U0.36 (PF7); no longer U0.38 (PF5)
- net row03: now also U0.25 (PD4); no longer U0.37 (PF6)
- net at ULED09.2 (DOUT): now also ULED10.4 (DIN)
- new net: ULED10.2 (DOUT), ULED11.4 (DIN)
Other:
- moved on the sheet: C3, C4, C5, C6, D00_00, D00_01, D00_02, D00_03, D01_00, D01_01, D01_02, D01_03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
